File: sciencefestivalpcb/sciencefestivalpcb.kicad_pcb (KiCad board)
At the start: 2 copper layers, 59 x 83 mm, 70 parts, among them IC1 RP402N331E-TR-FE, IC2 RP402N331E-TR-FE, J1 Conn_01x06_Pin, Q1 IRLTS6342TRPBF, Q2 IRLTS6342TRPBF, SW1 SW_SPST, U1 STM32L552CETx, U2 LSM6DSL

Commit message: Initial firmware commit
Changed lines of the file:
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@@
       (sketchpadsonfab false)
       (subtractmaskfromsilk false)
-      (outputformat 1)
+      (outputformat 4)
       (mirror false)
-      (drillshape 1)
+      (drillshape 0)
       (scaleselection 1)
       (outputdirectory "")
@@
     (fp_line (start 1 0.45) (end -1 0.45)
       (stroke (width 0.1) (type solid)) (layer "F.Fab"))
-    (pad "1" smd roundrect (at -1.15 0) (size 1.05 1.2) (layers "F.Cu" "F.Paste" "F.Mask") (roundrect_rratio 0.238095)
+    (pad "1" smd roundrect (at -1.15 0) (size 1.05 1.2) (layers "F.Cu" "F.Paste" "F.Mask") (roundrect_rratio 0.2380952381)
       (net 5 "Net-(IC2-LX)") (pinfunction "1") (pintype "passive"))
-    (pad "2" smd roundrect (at 1.15 0) (size 1.05 1.2) (layers "F.Cu" "F.Paste" "F.Mask") (roundrect_rratio 0.238095)
+    (pad "2" smd roundrect (at 1.15 0) (size 1.05 1.2) (layers "F.Cu" "F.Paste" "F.Mask") (roundrect_rratio 0.2380952381)
       (net 7 "VCC") (pinfunction "2") (pintype "passive"))
     (model "${KICAD6_3DMODEL_DIR}/Inductor_SMD.3dshapes/L_0805_2012Metric.wrl"
@@
     (pad "6" smd roundrect (at 3.125 -2.4 90) (size 0.8 1.6) (layers "F.Cu" "F.Paste" "F.Mask") (roundrect_rratio 0.25)
       (net 60 "/UART_TX") (pinfunction "Pin_6") (pintype "passive"))
-    (pad "MP" smd roundrect (at -5.675 0.5 90) (size 2.1 3) (layers "F.Cu" "F.Paste" "F.Mask") (roundrect_rratio 0.119048))
-    (pad "MP" smd roundrect (at 5.675 0.5 90) (size 2.1 3) (layers "F.Cu" "F.Paste" "F.Mask") (roundrect_rratio 0.119048))
+    (pad "MP" smd roundrect (at -5.675 0.5 90) (size 2.1 3) (layers "F.Cu" "F.Paste" "F.Mask") (roundrect_rratio 0.1190480952))
+    (pad "MP" smd roundrect (at 5.675 0.5 90) (size 2.1 3) (layers "F.Cu" "F.Paste" "F.Mask") (roundrect_rratio 0.1190480952))
     (model "${KICAD6_3DMODEL_DIR}/Connector_Molex.3dshapes/Molex_PicoBlade_53261-0671_1x06-1MP_P1.25mm_Horizontal.wrl"
       (offset (xyz 0 0 0))
@@
     (fp_line (start 1 0.45) (end -1 0.45)
       (stroke (width 0.1) (type solid)) (layer "F.Fab"))
-    (pad "1" smd roundrect (at -1.15 0) (size 1.05 1.2) (layers "F.Cu" "F.Paste" "F.Mask") (roundrect_rratio 0.238095)
+    (pad "1" smd roundrect (at -1.15 0) (size 1.05 1.2) (layers "F.Cu" "F.Paste" "F.Mask") (roundrect_rratio 0.2380952381)
       (net 4 "Net-(IC1-LX)") (pinfunction "1") (pintype "passive"))
-    (pad "2" smd roundrect (at 1.15 0) (size 1.05 1.2) (layers "F.Cu" "F.Paste" "F.Mask") (roundrect_rratio 0.238095)
+    (pad "2" smd roundrect (at 1.15 0) (size 1.05 1.2) (layers "F.Cu" "F.Paste" "F.Mask") (roundrect_rratio 0.2380952381)
       (net 7 "VCC") (pinfunction "2") (pintype "passive"))
     (model "${KICAD6_3DMODEL_DIR}/Inductor_SMD.3dshapes/L_0805_2012Metric.wrl"
@@
     (attr board_only exclude_from_pos_files exclude_from_bom)
     (fp_text reference "kibuzzard-65246046" (at 0 5.349734) (layer "B.SilkS") hide
-        (effects (font (size 0 0)) (justify mirror))
+        (effects (font (size 0 0) (thickness 0.15)) (justify mirror))
     )
     (fp_text value "G***" (at 0 -5.349734) (layer "B.SilkS") hide
-        (effects (font (size 0 0)) (justify mirror))
+        (effects (font (size 0 0) (thickness 0.15)) (justify mirror))
     )
     (fp_poly
@@
     (attr board_only exclude_from_pos_files exclude_from_bom)
     (fp_text reference "kibuzzard-65245FE4" (at 0 4.15925) (layer "B.SilkS") hide
-        (effects (font (size 0 0)) (justify mirror))
+        (effects (font (size 0 0) (thickness 0.15)) (justify mirror))
     )
     (fp_text value "G***" (at 0 -4.15925) (layer "B.SilkS") hide
-        (effects (font (size 0 0)) (justify mirror))
+        (effects (font (size 0 0) (thickness 0.15)) (justify mirror))
     )
     (fp_poly
@@
     (attr board_only exclude_from_pos_files exclude_from_bom)
     (fp_text reference "kibuzzard-652460C9" (at 0 4.417389) (layer "B.SilkS") hide
-        (effects (font (size 0 0)) (justify mirror))
+        (effects (font (size 0 0) (thickness 0.15)) (justify mirror))
     )
     (fp_text value "G***" (at 0 -4.417389) (layer "B.SilkS") hide
-        (effects (font (size 0 0)) (justify mirror))
+        (effects (font (size 0 0) (thickness 0.15)) (justify mirror))
     )
     (fp_poly
@@
     (attr board_only exclude_from_pos_files exclude_from_bom)
     (fp_text reference "kibuzzard-652460F9" (at 0 4.417389) (layer "B.SilkS") hide
-        (effects (font (size 0 0)) (justify mirror))
+        (effects (font (size 0 0) (thickness 0.15)) (justify mirror))
     )
     (fp_text value "G***" (at 0 -4.417389) (layer "B.SilkS") hide
-        (effects (font (size 0 0)) (justify mirror))
+        (effects (font (size 0 0) (thickness 0.15)) (justify mirror))
     )
     (fp_poly
@@
     (attr board_only exclude_from_pos_files exclude_from_bom)
     (fp_text reference "kibuzzard-652460F2" (at 0 3.630083) (layer "B.SilkS") hide
-        (effects (font (size 0 0)) (justify mirror))
+        (effects (font (size 0 0) (thickness 0.15)) (justify mirror))
     )
     (fp_text value "G***" (at 0 -3.630083) (layer "B.SilkS") hide
-        (effects (font (size 0 0)) (justify mirror))
+        (effects (font (size 0 0) (thickness 0.15)) (justify mirror))
     )
     (fp_poly
@@
     (attr board_only exclude_from_pos_files exclude_from_bom)
     (fp_text reference "kibuzzard-652460E7" (at 0 4.417389) (layer "B.SilkS") hide
-        (effects (font (size 0 0)) (justify mirror))
+        (effects (font (size 0 0) (thickness 0.15)) (justify mirror))
     )
     (fp_text value "G***" (at 0 -4.417389) (layer "B.SilkS") hide
-        (effects (font (size 0 0)) (justify mirror))
+        (effects (font (size 0 0) (thickness 0.15)) (justify mirror))
     )
     (fp_poly
