File: sciencefestivalpcb/sciencefestivalpcb.kicad_sch (KiCad schematic)
At the start: 63 parts, among them IC1 RP402N331E-TR-FE, IC2 RP402N331E-TR-FE, J1 Conn_01x06_Pin, Q1 IRLTS6342TRPBF, Q2 IRLTS6342TRPBF, SW1 SW_SPST, U1 STM32L552CETx, U2 LSM6DSL

Commit message: Initial firmware commit
Parts:
- BZ1: Mouser Price/Stock (none) -> https://nl.mouser.com/ProductDetail/CUI-Devices/CSQG703BP?q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; Price (none) -> 0.772
- C1, C2, C3, C4: MPN GRM188R60J106ME47 -> 06033D106KAT2A; Mouser Price/Stock (none) -> https://nl.mouser.com/ProductDetail/KYOCERA-AVX/06033D106KA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; Price (none) -> 0.19
- C10, C12, C5, C6, C7, C8, C9: MPN (none) -> GRJ188R72A104KE11D; Mouser Price/Stock (none) -> https://nl.mouser.com/ProductDetail/Murata-Electronics/GRJ1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; Price (none) -> 0.05
- C11: MPN (none) -> GRM188R6YA475KE15D; Mouser Price/Stock (none) -> https://nl.mouser.com/ProductDetail/Murata-Electronics/GRM1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; Price (none) -> 0.19
- C13: MPN (none) -> 06033W105KAT2A; Mouser Price/Stock (none) -> https://nl.mouser.com/ProductDetail/KYOCERA-AVX/06033W105KA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; Price (none) -> 0.143
- D1, D2, D3, D4, D5, D6, D7: MPN IN-PI554FCH -> IN-PI554FCH; Mouser Price/Stock (none) -> https://nl.mouser.com/ProductDetail/Inolux/IN-PI554FCH?qs=f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; Price (none) -> 0.436
- D10, D8, D9: Mouser Price/Stock (none) -> https://nl.mouser.com/ProductDetail/ROHM-Semiconductor/SMLV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; Price (none) -> 0.93
- H1: MPN (none) -> BAT-HLD-003-SMT; Mouser Price/Stock (none) -> https://nl.mouser.com/ProductDetail/TE-Connectivity-Linx-Te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; Price (none) -> 0.446
- IC1: MPN (none) -> RP402N331E-TR-FE; Price (none) -> 1.49
- IC2: MPN (none) -> RP402N501E-TR-FE; Mouser Price/Stock https://www.mouser.co.uk/ProductDetail/Nisshinbo/RP402N331E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 -> https://nl.mouser.com/ProductDetail/Nisshinbo/RP402N501E-TR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; Price (none) -> 1.52
- J1: MPN (none) -> 53261-0671; Mouser Price/Stock (none) -> https://nl.mouser.com/ProductDetail/Molex/53261-0671?qs=%25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
- L1, L2: Mouser Price/Stock (none) -> https://nl.mouser.com/ProductDetail/Vishay-Dale/IHHP0805ZHE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; Price (none) -> 0.261
- Q1, Q2: MPN (none) -> IRLTS6342TRPBF; Price (none) -> 0.372
- R1, R4, R7: MPN (none) -> ERJ-UP3J331V; Mouser Price/Stock (none) -> https://nl.mouser.com/ProductDetail/Panasonic/ERJ-UP3J331V?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; Price (none) -> 0.028
- R12, R13, R14: MPN (none) -> ERJ-3GEY0R00V; Mouser Price/Stock (none) -> https://nl.mouser.com/ProductDetail/Panasonic/ERJ-3GEY0R00V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; Price (none) -> 0.009
- R2, R3, R5, R6, R8, R9: MPN (none) -> ERJ-UP3F5100V; Mouser Price/Stock (none) -> https://nl.mouser.com/ProductDetail/Panasonic/ERJ-UP3F5100V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; Price (none) -> 0.041
- SW1: Mouser Price/Stock (none) -> https://nl.mouser.com/ProductDetail/Omron-Electronics/A6S-1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; Price (none) -> 1.65
- U1: Mouser Price/Stock (none) -> https://nl.mouser.com/ProductDetail/STMicroelectronics/STM3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; Price (none) -> 9.77
- U2: Mouser Price/Stock (none) -> https://nl.mouser.com/ProductDetail/STMicroelectronics/LSM6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; Price (none) -> 5.67
